Commit message: Completed protoype car model in Rviz2

File: description/robot.urdf.xacro (robot description, xacro)
@@ -2,7 +2,3 @@
 <robot xmlns:xacro="http://www.ros.org/wiki/xacro"  name="robot">
     <xacro:include filename="robot_core.xacro" />
-    <!--
-    <link name="base_link">
-    </link>
-    -->
 </robot>

File: description/robot_core.xacro (robot description, xacro)
@@ -1,7 +1,10 @@
 <?xml version="1.0"?>
 <robot xmlns:xacro="http://www.ros.org/wiki/xacro"  >
-   <xacro:include filename="robot_colors.xacro" />
+    <xacro:include filename="robot_colors.xacro" />
+    <xacro:include filename="inertial_macros.xacro" />
+    <!-- BASE LINK -->
     <link name="base_link">
     </link>
+    <!-- CHASSIS -->
     <joint name="chassis_joint" type="fixed">
         <parent link="base_link"/>
@@ -15,6 +18,88 @@
                 <box size="0.461 0.311 0.178"/>
             </geometry>
+            <material name="white"/>
+        </visual>
+        <collision>
+            <origin xyz="0.2305 0 0.089" rpy="0 0 0"/>
+            <geometry>
+                <box size="0.461 0.311 0.178"/>
+            </geometry>
+        </collision>
+        <xacro:inertial_box mass="1.69" x="0.461" y="0.311" z="0.178">
+            <origin xyz="0.2305 0 0.089" rpy="0 0 0"/>
+        </xacro:inertial_box>
+    </link>
+    <!-- LEFT DRIVE WHEEL  -->
+    <joint name="left_wheel_joint" type="continuous">
+        <parent link="base_link"/>
+        <child link="left_wheel"/>
+        <origin xyz="0 0.175 0" rpy="-${pi/2} 0 0"/>
+        <axis xyz="0 0 1"/>
+    </joint>
+    <link name="left_wheel">
+        <visual>
+            <geometry>
+                <cylinder length="0.04" radius="0.05" />
+            </geometry>
             <material name="orange"/>
         </visual>
+        <collision>
+            <geometry>
+                <cylinder length="0.04" radius="0.05" />
+            </geometry>
+        </collision>
+        <!--NEED TO MEASURE PARAMETERS FOR WHEELS AND UPDATE-->
+        <xacro:inertial_cylinder mass="0.1" length="0.04" radius="0.05">
+            <origin xyz="0 0 0" rpy="0 0 0"/>
+        </xacro:inertial_cylinder>
+    </link>
+    <!-- RIGHT DRIVE WHEEL -->
+    <joint name="right_wheel_joint" type="continuous">
+        <parent link="base_link"/>
+        <child link="right_wheel"/>
+        <origin xyz="0 -0.175 0" rpy="${pi/2} 0 0"/>
+        <axis xyz="0 0 -1"/>
+    </joint>
+    <link name="right_wheel">
+        <visual>
+            <geometry>
+                <cylinder length="0.04" radius="0.05" />
+            </geometry>
+            <material name="orange"/>
+        </visual>
+        <collision>
+            <geometry>
+                <cylinder length="0.04" radius="0.05" />
+            </geometry>
+        </collision>
+        <!--NEED TO MEASURE PARAMETERS FOR WHEELS AND UPDATE-->
+        <xacro:inertial_cylinder mass="0.1" length="0.04" radius="0.05">
+            <origin xyz="0 0 0" rpy="0 0 0"/>
+        </xacro:inertial_cylinder>
+    </link>
+    <!-- CASTER WHEEL -->
+    <!-- CREATE TWO CASTER WHEELS LATER-->
+    <joint name="caster_wheel_joint" type="fixed">
+        <parent link="chassis"/>
+        <child link="caster_wheel"/>
+        <origin xyz="0.24 0 0" rpy="0 0 0"/>
+    </joint>
+    <!--UPDATE THIS TO CYLINDER ONCE PARAMETERS FOR WHEELS IS MEASURED-->
+    <link name="caster_wheel">
+        <visual>
+            <geometry>
+                <sphere radius="0.05" />
+            </geometry>
+            <material name="orange"/>
+        </visual>
+        <collision>
+            <geometry>
+                <sphere radius="0.05" />
+            </geometry>
+        </collision>
+        <!--UPDATE THIS TO CYLINDER ONCE PARAMETERS FOR WHEELS IS MEASURED-->
+        <xacro:inertial_sphere mass="0.1" radius="0.05">
+            <origin xyz="0 0 0" rpy="0 0 0"/>
+        </xacro:inertial_sphere>
     </link>
 </robot>

Commit message: updated ackermann controller and robot description

File: description/robot.urdf.xacro (robot description, xacro)
@@ -2,3 +2,4 @@
 <robot xmlns:xacro="http://www.ros.org/wiki/xacro"  name="robot">
     <xacro:include filename="robot_core.xacro" />
+    <xacro:include filename="ros2_ack.xacro" />
 </robot>

File: description/robot_core.xacro (robot description, xacro)
@@ -4,5 +4,5 @@
     <xacro:property name="wheel_radius" value="${$(arg wheel_diameter)/2}"/>
     <xacro:property name="wheel_width" value="0.047"/>
-    <xacro:property name="wheel_friction" value="0.8"/>
+    <xacro:property name="wheel_friction" value="0.01"/>
     <xacro:property name="wheelbase_length" value="0.311"/>
     <xacro:property name="front_wheelbase_width" value="0.289"/>
@@ -35,30 +35,5 @@
         </inertial>
     </xacro:macro>
-    <link name="base_footprint"/>
     <link name="base_link"/>
-    <!--
-    <link name="base_link">
-        <visual>
-        <origin xyz="0 0 0.1" rpy="0 0 0"/>
-        <geometry>
-            <cylinder length="0.2" radius="0.01"/>
-        </geometry>
-        <material name="silver">
-            <color rgba="0.75 0.75 0.75 1"/>
-        </material>
-        </visual>
-        <collision>
-        <origin xyz="0 0 0.1" rpy="0 0 0"/>
-        <geometry>
-            <cylinder length="0.2" radius="0.01"/>
-        </geometry>
-        </collision>
-        <inertial>
-        <mass value="0.01"/>
-        <inertia ixx="0.015" iyy="0.0375" izz="0.0375"
-                ixy="0" ixz="0" iyz="0"/>
-        </inertial>
-    </link>
-    -->
     <link name="chassis_link">
         <visual>
@@ -317,9 +292,9 @@
         </inertial>
     </link>
-    <joint name="base_link_joint" type="fixed">
+<!--    <joint name="base_link_joint" type="fixed">
         <parent link="base_footprint"/>
         <child link="base_link"/>
         <origin rpy="0 0 0" xyz="0 0 0"/>
-    </joint>
+    </joint>-->
     <joint name="laser_scanner_joint" type="fixed">
         <origin rpy="0 0 0" xyz="0.1397 0 0.2159"/>
@@ -402,17 +377,17 @@
     <gazebo reference="front_left_wheel">
         <mu1>${wheel_friction}</mu1>
-        <material>Gazebo/DarkGrey</material>
+        <material>Gazebo/Black</material>
     </gazebo>
     <gazebo reference="front_right_wheel">
         <mu1>${wheel_friction}</mu1>
-        <material>Gazebo/DarkGrey</material>
+        <material>Gazebo/Black</material>
     </gazebo>
     <gazebo reference="back_left_wheel">
         <mu1>${wheel_friction}</mu1>
-        <material>Gazebo/DarkGrey</material>
+        <material>Gazebo/Green</material>
     </gazebo>
     <gazebo reference="back_right_wheel">
         <mu1>${wheel_friction}</mu1>
-        <material>Gazebo/DarkGrey</material>
+        <material>Gazebo/Green</material>
     </gazebo>
     <gazebo reference="base_link">
@@ -423,3 +398,3 @@
         </plugin>
     </gazebo>
-    </robot>
+</robot>

File: description/robot_core_f1tenth.xacro (robot description, xacro)
@@ -3,7 +3,6 @@
     <xacro:include filename="robot_colors.xacro" />
     <xacro:include filename="inertial_macros.xacro" />
-    <xacro:include filename="ros2_ack.xacro"/>
-    <xacro:property name="wheelbase" value="0.289" />
-    <xacro:property name="width" value="0.311" />
+    <xacro:property name="wheelbase" value="0.311" />
+    <xacro:property name="width" value="0.289" />
     <xacro:property name="height" value="0.178" />
     <xacro:property name="ground_offset" value="0.04" /> <!--Measure this-->
@@ -44,9 +43,15 @@
     <link name="laser_model">
         <visual>
-        <geometry>
-            <cylinder radius="${laser_radius}" length="${laser_height}"/>
-        </geometry>
-        <material name="black"/>
-        </visual>
+            <geometry>
+                <cylinder radius="${laser_radius}" length="${laser_height}"/>
+            </geometry>
+            <material name="black"/>
+        </visual>
+        <collision>
+            <geometry>
+                <cylinder radius="${laser_radius}" length="${laser_height}"/>
+            </geometry>
+            <material name="black"/>
+        </collision>
     </link>
     <gazebo reference="laser_model">
@@ -118,17 +123,15 @@
 		<visual>
             <geometry>
-                <cylinder radius="0.02" length="0.04"/>
-            </geometry>
-            <material name="blue"/>
-            <origin xyz="0 0 0" rpy="${pi/2} 0 0"/>
+                <cylinder radius="0.01" length="0.01"/>
+            </geometry>
+            <material name="blue"/>
 		</visual>
         <collision>
             <geometry>
-                <cylinder radius="0.02" length="0.04"/>
-            </geometry>
-            <material name="blue"/>
-            <origin xyz="0 0 0" rpy="${pi/2} 0 0"/>
-        </collision>
-        <xacro:inertial_cylinder mass="0.1" length="0.04" radius="0.02">
+                <cylinder radius="0.01" length="0.04"/>
+            </geometry>
+            <material name="blue"/>
+        </collision>
+        <xacro:inertial_cylinder mass="0.1" length="0.04" radius="0.01">
             <origin xyz="0 0 0" rpy="0 0 0"/>
         </xacro:inertial_cylinder>
@@ -172,20 +175,18 @@
     </joint>
     <link name="front_right_hinge">
-    	<visual>
-            <geometry>
-                <cylinder radius="0.02" length="0.04"/>
-            </geometry>
-            <material name="blue"/>
-            <origin xyz="${wheelbase} 0 0" rpy="${pi/2} 0 0"/>
+		<visual>
+            <geometry>
+                <cylinder radius="0.01" length="0.01"/>
+            </geometry>
+            <material name="blue"/>
 		</visual>
         <collision>
             <geometry>
-                <cylinder radius="0.02" length="0.04"/>
-            </geometry>
-            <material name="blue"/>
-            <origin xyz="${wheelbase} 0 0" rpy="${pi/2} 0 0"/>
-        </collision>
-        <xacro:inertial_cylinder mass="0.1" length="0.04" radius="0.02">
-            <origin xyz="${wheelbase} 0 0" rpy="${pi/2} 0 0"/>
+                <cylinder radius="0.01" length="0.04"/>
+            </geometry>
+            <material name="blue"/>
+        </collision>
+        <xacro:inertial_cylinder mass="0.1" length="0.04" radius="0.01">
+            <origin xyz="0 0 0" rpy="0 0 0"/>
         </xacro:inertial_cylinder>
     </link>

File: description/ros2_ack.xacro (robot description, xacro)
@@ -4,28 +4,22 @@
         <hardware>
             <plugin>gazebo_ros2_control/GazeboSystem</plugin>
-            <!--
-            <plugin>ros2_control_demo_example_11/CarlikeBotSystemHardware</plugin>
-            <param name="example_param_hw_start_duration_sec">0</param>
-            <param name="example_param_hw_stop_duration_sec">3.0</param>
-            <param name="is_simulation">1</param>
-            -->
         </hardware>
         <!-- Front Left Wheel Steer-->
-        <joint name="front_left_hinge_joint">
+        <joint name="front_left_wheel_steer_joint">
             <command_interface name="position"/>
             <state_interface name="position" />
         </joint>
         <!-- Front Right Wheel Steer-->
-        <joint name="front_right_hinge_joint">
+        <joint name="front_right_wheel_steer_joint">
           <command_interface name="position"/>
           <state_interface name="position" />
         </joint>
         <!-- Rear Left Wheel Drive-->
-        <joint name="base_to_back_left_wheel">
+        <joint name="back_left_wheel_joint">
             <command_interface name="velocity"/>
             <state_interface name="velocity" />
         </joint>
         <!-- Rear Right Wheel Drive-->
-        <joint name="base_to_back_right_wheel">
+        <joint name="back_right_wheel_joint">
             <command_interface name="velocity"/>
             <state_interface name="velocity" />
@@ -34,12 +28,10 @@
     <gazebo>
         <plugin filename="libgazebo_ros2_control.so" name="gazebo_ros2_control">
-            <!--
             <ros>
-                <remapping>asc/reference_unstamped:=cmd_vel</remapping>
+                <remapping>asc/reference:=cmd_vel</remapping>
                 <remapping>asc/odometry:=odom</remapping>
                 <remapping>asc/tf_odometry:=tf</remapping>
             </ros>
-            -->
-            <parameters>$(find team6_car)/config/controller/my_controllers.yaml</parameters>
+            <parameters>$(find team6_car)/config/my_controllers.yaml</parameters>
         </plugin>
     </gazebo>
