Commit message: Converted to bicycle steering and added microROS hardware interface for ros_control

File: description/robot.urdf.xacro (robot description, xacro)
@@ -1,5 +1,8 @@
 <?xml version="1.0"?>
 <robot xmlns:xacro="http://www.ros.org/wiki/xacro"  name="robot">
+    <xacro:include filename="inertial_macros.xacro" />
+    <xacro:include filename="materials.xacro" />
+    <xacro:include filename="lidar.xacro" />
     <xacro:include filename="robot_core.xacro" />
-    <xacro:include filename="ros2_ack.xacro" />
+    <xacro:include filename="ros2_bicycle.xacro" />
 </robot>

File: description/robot_core.xacro (robot description, xacro)
@@ -1,400 +1,253 @@
 <?xml version="1.0"?>
-<robot xmlns:xacro="http://ros.org/wiki/xacro" name="car">
-    <xacro:arg name="wheel_diameter" default="0.14224"/>
-    <xacro:property name="wheel_radius" value="${$(arg wheel_diameter)/2}"/>
-    <xacro:property name="wheel_width" value="0.047"/>
-    <xacro:property name="wheel_friction" value="0.01"/>
-    <xacro:property name="wheelbase_length" value="0.311"/>
-    <xacro:property name="front_wheelbase_width" value="0.289"/>
-    <xacro:property name="rear_wheelbase_width" value="0.289"/>
-    <xacro:property name="wheel_mass" value="0.1"/>
-    <xacro:property name="total_mass" value = "3.0"/>
-    <xacro:property name="shock_travel" value = "0.09"/>
-    <xacro:property name="chassis_height" value = "0.178"/>
-    <xacro:property name="chassis_elevation" value = "-0.01"/>
-    <xacro:property name="chassis_mass" value = "${total_mass-4*wheel_mass}"/>
-    <xacro:macro name="cylinder_inertia" params="m r h">
-            <inertia  ixx="${m*(3*r*r+h*h)/12}" ixy = "0" ixz = "0"
-                        iyy="${m*(3*r*r+h*h)/12}" iyz = "0"
-                        izz="${m*r*r/2}" />
-    </xacro:macro>
-    <xacro:macro name="box_inertia" params="m x y z">
-            <inertia  ixx="${m*(y*y+z*z)/12}" ixy = "0" ixz = "0"
-                        iyy="${m*(x*x+z*z)/12}" iyz = "0"
-                        izz="${m*(x*x+z*z)/12}" />
-    </xacro:macro>
-    <xacro:macro name="sphere_inertia" params="m r">
-            <inertia  ixx="${2*m*r*r/5}" ixy = "0" ixz = "0"
-                        iyy="${2*m*r*r/5}" iyz = "0"
-                        izz="${2*m*r*r/5}" />
-    </xacro:macro>
-    <xacro:macro name="cylinder_inertial" params="m r h">
-        <inertial>
-        <mass value="${m}"/>
-        <xacro:cylinder_inertia m="${m}" r="${r}" h="${h}"/>
-        </inertial>
-    </xacro:macro>
-    <link name="base_link"/>
-    <link name="chassis_link">
-        <visual>
-        <geometry>
-            <box size="${wheelbase_length} ${front_wheelbase_width} ${chassis_height}"/>
-        </geometry>
-        </visual>
+<robot xmlns:xacro="http://www.ros.org/wiki/xacro">
+  <!-- Constants for robot dimensions -->
+  <xacro:property name="PI" value="3.1415926535897931"/>
+  <xacro:property name="base_mass" value="4.0" /> <!-- arbitrary value for base mass -->
+  <xacro:property name="base_width" value="0.260" />
+  <xacro:property name="base_length" value="0.525" />
+  <xacro:property name="base_height" value="0.060" />
+  <xacro:property name="wheelbase" value="0.325" />
+  <xacro:property name="wheel_mass" value="0.34055" /> <!-- arbitrary value for wheel mass -->
+  <xacro:property name="wheel_len" value="0.045" />
+  <xacro:property name="wheel_radius" value="0.05" />
+  <!-- <xacro:property name="wheeltrack" value="" -->
+  <!-- Base Link -->
+  <link name="base_link" />
+  <!-- Chassis -->
+  <link name="chassis_link">
+    <collision>
+      <origin xyz="0 0 0" rpy="0 0 0"/>
+      <geometry>
+        <box size="${base_length} ${base_width} ${base_height}"/>
+      </geometry>
+    </collision>
+    <visual>
+      <origin xyz="0 0 0" rpy="0 0 0"/>
+      <geometry>
+        <box size="${base_length} ${base_width} ${base_height}"/>
+      </geometry>
+      <material name="orange"/>
+    </visual>
+    <!-- <inertial>
+      <origin xyz="0 0 0" rpy="0 0 0"/>
+      <mass value="${base_mass}"/>
+        <inertia
+          ixx="0.000270" ixy="0.0" ixz="0.0"
+          iyy="0.000270" iyz="0.0"
+          izz="0.000426"/>
+      </inertial> -->
+    <xacro:inertial_box mass="${base_mass}" x="${wheelbase}" y="${base_width}" z="${base_height}">
+      <origin xyz="0 0 0" rpy="0 0 0"/>
+    </xacro:inertial_box>
+    </link>
+    <gazebo reference="chassis_link">
+        <material>Gazebo/Black</material>
+    </gazebo>
+    <joint name="chassis_joint" type="fixed">
+      <parent link="base_link"/>
+      <child link="chassis_link"/>
+      <origin xyz="0 0 ${base_height/2 + wheel_radius}" rpy="0 0 0"/>
+      <axis xyz="0 0 1"/>
+      <dynamics damping="0.2"/>
+    </joint>
+    <!-- rear wheels -->
+    <!-- virtual rear wheel -->
+    <link name="virtual_rear_wheel">
+      <visual>
+        <origin xyz="0 0 0" rpy="${PI/2} 0 ${PI/2}"/>
+        <geometry>
+          <cylinder length="0.01" radius="${wheel_radius}"/>
+        </geometry>
+        <material name="invisible"/>
+      </visual>
+    </link>
+    <gazebo reference="virtual_rear_wheel">
+        <material>Gazebo/White</material>
+    </gazebo>
+    <joint name="virtual_rear_wheel_joint" type="continuous">
+      <parent link="chassis_link"/>
+      <child link="virtual_rear_wheel"/>
+      <origin xyz="-${wheelbase/2} 0 -${base_height/2}" rpy="0 0 ${PI/2}"/>
+      <axis xyz="1 0 0"/>
+      <limit effort="100.0" velocity="100.0"/>
+      <dynamics damping="0.2"/>
+    </joint>
+    <!-- rear right wheel -->
+    <link name="rear_right_wheel">
+      <collision>
+        <origin xyz="0 0 0" rpy="${PI/2} 0 ${PI/2}"/>
+        <geometry>
+          <cylinder length="${wheel_len}" radius="${wheel_radius}"/>
+        </geometry>
+      </collision>
+      <visual>
+        <origin xyz="0 0 0" rpy="${PI/2} 0 ${PI/2}"/>
+        <geometry>
+          <cylinder length="${wheel_len}" radius="${wheel_radius}"/>
+        </geometry>
+        <material name="black"/>
+      </visual>
+      <!-- <inertial>
+        <origin xyz="0 0 0" rpy="${PI/2} 0 ${PI/2}"/>
+        <mass value="${wheel_mass}"/>
+        <inertia
+          ixx="0.000270" ixy="0.0" ixz="0.0"
+          iyy="0.000270" iyz="0.0"
+          izz="0.000426"/>
+      </inertial> -->
+      <xacro:inertial_cylinder mass="${wheel_mass}" length="${wheel_len}" radius="${wheel_radius}">
+          <origin xyz="0 0 0" rpy="${PI/2} 0 ${PI/2}"/>
+      </xacro:inertial_cylinder>
+    </link>
+    <gazebo reference="rear_right_wheel">
+        <material>Gazebo/Orange</material>
+    </gazebo>
+    <joint name="rear_right_wheel_joint" type="continuous">
+      <parent link="chassis_link"/>
+      <child link="rear_right_wheel"/>
+      <origin xyz="-${wheelbase/2} ${base_width/2} -${base_height/2}" rpy="0 0 ${PI/2}"/>
+      <axis xyz="1 0 0"/>
+      <limit effort="100.0" velocity="100.0"/>
+      <dynamics damping="0.2"/>
+      <mimic joint="virtual_rear_wheel_joint" multiplier="1.0" offset="0.0"/>
+    </joint>
+    <!-- rear left wheel -->
+    <link name="rear_left_wheel">
         <collision>
-        <geometry>
-            <box size="${wheelbase_length} ${front_wheelbase_width} ${chassis_height}"/>
-        </geometry>
-        </collision>
-        <inertial>
-        <mass value="${chassis_mass}"/>
-        <xacro:box_inertia m="${chassis_mass}" x="${wheelbase_length}" y="${front_wheelbase_width}" z="${chassis_height}"/>
-        </inertial>
-    </link>
-    <link name="back_left_wheel">
-        <visual>
-        <geometry>
-            <cylinder length="${wheel_width}" radius="${wheel_radius}"/>
-        </geometry>
-        <material name="black">
-            <color rgba="0 0 0 1"/>
-        </material>
-        </visual>
-        <collision>
-        <geometry>
-            <cylinder length="${wheel_width}" radius="${wheel_radius}"/>
-        </geometry>
-        </collision>
-        <xacro:cylinder_inertial m="${wheel_mass}" r="${wheel_radius}" h="${wheel_width}"/>
-    </link>
-    <link name="laser_scanner_link">
-        <collision>
-        <origin xyz="0 0 0" rpy="0 0 0"/>
-        <geometry>
-            <box size=".127 0.1016 0.0508"/>
-        </geometry>
+          <origin xyz="0 0 0" rpy="${PI/2} 0 ${PI/2}"/>
+          <geometry>
+            <cylinder length="${wheel_len}" radius="${wheel_radius}"/>
+          </geometry>
         </collision>
         <visual>
-        <origin xyz="0 0 0" rpy="0 0 0"/>
-        <geometry>
-            <box size=".127 0.1016 0.0508"/>
-        </geometry>
+          <origin xyz="0 0 0" rpy="${PI/2} 0 ${PI/2}"/>
+          <geometry>
+            <cylinder length="${wheel_len}" radius="${wheel_radius}"/>
+          </geometry>
+          <material name="black"/>
         </visual>
-        <inertial>
-        <mass value="1e-5"/>
-        <origin xyz="0 0 0" rpy="0 0 0"/>
-        <inertia ixx="1e-6" ixy="0" ixz="0" iyy="1e-6" iyz="0" izz="1e-6"/>
-        </inertial>
-    </link>
-    <gazebo reference="laser_scanner_link">
-        <sensor type="ray" name="laser_scanner">
-        <always_on>true</always_on>
-        <!-- <visualize>true</visualize> -->
-        <update_rate>3</update_rate>
-        <ray>
-        <scan>
-            <horizontal>
-            <samples>360</samples>
-            <resolution>1</resolution>
-            <min_angle>${-pi}</min_angle>
-            <max_angle>${pi}</max_angle>
-            </horizontal>
-        </scan>
-        <range>
-            <min>0.30</min>
-            <max>25.0</max>
-            <resolution>0.1</resolution>
-        </range>
-        </ray>
-        <plugin name="scan" filename="libgazebo_ros_ray_sensor.so">
-            <ros>
-            <remapping>~/out:=scan</remapping>
-            </ros>
-            <output_type>sensor_msgs/LaserScan</output_type>
-            <frame_name>laser_scanner_link</frame_name>
-        </plugin>
-        </sensor>
-    </gazebo>
-    <link name="back_right_wheel">
-        <visual>
-        <geometry>
-            <cylinder length="${wheel_width}" radius="${wheel_radius}"/>
-        </geometry>
-        <material name="black">
-            <color rgba="0 0 0 1"/>
-        </material>
-        </visual>
-        <collision>
-        <geometry>
-            <cylinder length="${wheel_width}" radius="${wheel_radius}"/>
-        </geometry>
-        </collision>
-        <xacro:cylinder_inertial m="${wheel_mass}" r="${wheel_radius}" h="${wheel_width}"/>
-    </link>
-    <link name="front_left_wheel_steer">
-        <visual>
-        <geometry>
-            <cylinder length="0.01" radius="0.01"/>
-        </geometry>
-        <material name="black">
-            <color rgba="0 0 0 1"/>
-        </material>
-        </visual>
-        <collision>
-        <geometry>
-            <cylinder length="0.01" radius="0.01"/>
-        </geometry>
-        </collision>
-        <inertial>
-        <mass value="0.1"/>
-        <inertia ixx="5.1458e-5" iyy="5.1458e-5" izz="6.125e-5"
-                ixy="0" ixz="0" iyz="0"/>
-        </inertial>
-    </link>
-        <link name="front_left_wheel">
-        <visual>
-        <geometry>
-            <cylinder length="${wheel_width}" radius="${wheel_radius}"/>
-        </geometry>
-        <material name="black">
-            <color rgba="0 0 0 1"/>
-        </material>
-        </visual>
-        <collision>
-        <geometry>
-            <cylinder length="${wheel_width}" radius="${wheel_radius}"/>
-        </geometry>
-        </collision>
-        <xacro:cylinder_inertial m="${wheel_mass}" r="${wheel_radius}" h="${wheel_width}"/>
-    </link>
-    <link name="front_right_wheel_steer">
-        <visual>
-        <geometry>
-            <cylinder length="0.01" radius="0.01"/>
-        </geometry>
-        <material name="black">
-            <color rgba="0 0 0 1"/>
-        </material>
-        </visual>
-        <collision>
-        <geometry>
-            <cylinder length="0.01" radius="0.01"/>
-        </geometry>
-        </collision>
-        <inertial>
-        <mass value="0.1"/>
-        <inertia ixx="5.1458e-5" iyy="5.1458e-5" izz="6.125e-5"
-                ixy="0" ixz="0" iyz="0"/>
-        </inertial>
-    </link>
+        <!-- <inertial>
+          <origin xyz="0 0 0" rpy="${PI/2} 0 ${PI/2}"/>
+          <mass value="${wheel_mass}"/>
+          <inertia
+            ixx="0.000270" ixy="0.0" ixz="0.0"
+            iyy="0.000270" iyz="0.0"
+            izz="0.000426"/>
+        </inertial> -->
+      <xacro:inertial_cylinder mass="${wheel_mass}" length="${wheel_len}" radius="${wheel_radius}">
+          <origin xyz="0 0 0" rpy="${PI/2} 0 ${PI/2}"/>
+      </xacro:inertial_cylinder>
+    </link>
+    <gazebo reference="rear_left_wheel">
+        <material>Gazebo/Orange</material>
+    </gazebo>
+    <joint name="rear_left_wheel_joint" type="continuous">
+      <parent link="chassis_link" />
+      <child link="rear_left_wheel" />
+      <origin xyz="-${wheelbase/2} -${base_width/2} -${base_height/2}" rpy="0 0 ${PI/2}"/>
+      <axis xyz="1 0 0"/>
+      <limit effort="100.0" velocity="100.0"/>
+      <dynamics damping="0.2"/>
+      <mimic joint="virtual_rear_wheel_joint" multiplier="1.0" offset="0.0"/>
+    </joint>
+    <!-- front wheels -->
+    <!-- virtual front wheel -->
+    <link name="virtual_front_wheel">
+      <visual>
+        <origin xyz="0 0 0" rpy="${PI/2} 0 ${PI/2}"/>
+        <geometry>
+          <cylinder length="0.01" radius="${wheel_radius}"/>
+        </geometry>
+        <material name="invisible"/>
+      </visual>
+    </link>
+    <gazebo reference="virtual_front_wheel">
+        <material>Gazebo/Black</material>
+    </gazebo>
+    <joint name="virtual_front_wheel_joint" type="revolute">
+      <parent link="chassis_link"/>
+      <child link="virtual_front_wheel"/>
+      <origin xyz="${wheelbase/2} 0 -${base_height/2}" rpy="0 0 ${PI/2}"/>
+      <axis xyz="0 0 1"/>
+      <limit lower="-0.4" upper="0.4" effort="100.0" velocity="0.0"/>
+      <dynamics damping="0.2"/>
+    </joint>
+    <!-- front right wheel -->
     <link name="front_right_wheel">
-        <visual>
-        <geometry>
-            <cylinder length="${wheel_width}" radius="${wheel_radius}"/>
-        </geometry>
-        <material name="black">
-            <color rgba="0 0 0 1"/>
-        </material>
-        </visual>
-        <collision>
-        <geometry>
-            <cylinder length="${wheel_width}" radius="${wheel_radius}"/>
-        </geometry>
-        </collision>
-        <xacro:cylinder_inertial m="${wheel_mass}" r="${wheel_radius}" h="${wheel_width}"/>
-    </link>
-    <link name="back_left_wheel_shock">
-        <visual>
-        <origin xyz="0 0 0.1" rpy="0 0 0"/>
-        <geometry>
-            <cylinder length="0.05" radius="0.01"/>
-        </geometry>
-        <material name="silver">
-            <color rgba="0.75 0.75 0.75 1"/>
-        </material>
-        </visual>
-        <collision>
-        <origin xyz="0 0 0.1" rpy="0 0 0"/>
-        <geometry>
-            <cylinder length="0.05" radius="0.01"/>
-        </geometry>
-        </collision>
-        <inertial>
-        <mass value="0.01"/>
-        <inertia ixx="0.015" iyy="0.0375" izz="0.0375"
-                ixy="0" ixz="0" iyz="0"/>
-        </inertial>
-    </link>
-    <link name="back_right_wheel_shock">
-        <visual>
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