Commit message: Added translations for twist to PWM

File: description/ros2_bicycle.xacro (robot description, xacro)
@@ -1,18 +1,23 @@
 <?xml version="1.0"?>
 <robot xmlns:xacro="http://www.ros.org/wiki/xacro">
-    <ros2_control name="RealRobot" type="system">
-        <hardware>
-          <plugin>real_car/RealCarHardware</plugin>
-        </hardware>
-      <joint name="virtual_front_wheel_joint">
-        <command_interface name="position"/>
-        <state_interface name="position"/>
-      </joint>
-      <joint name="virtual_rear_wheel_joint">
-        <command_interface name="velocity"/>
-        <state_interface name="velocity"/>
-        <state_interface name="position"/>
-      </joint>
-    </ros2_control>
+  <ros2_control name="RealRobot" type="system">
+    <hardware>
+      <plugin>real_car/RealCarHardware</plugin>
+    </hardware>
+    <joint name="virtual_front_wheel_joint">
+      <command_interface name="position"/>
+        <param name = "min">-1</param>
+        <param name = "max">1</param>
+      <state_interface name="position"/>
+    </joint>
+    <joint name="virtual_rear_wheel_joint">
+      <command_interface name="velocity">
+        <param name = "min">-1</param>
+        <param name = "max">1</param>
+      </command_interface>
+      <state_interface name="velocity"/>
+      <state_interface name="position"/>
+    </joint>
+  </ros2_control>
 <!--     <gazebo>
         <plugin name="gazebo_ros2_control" filename="libgazebo_ros2_control.so">
