Commit message: new

File: description/lidar.xacro (robot description, xacro)
@@ -4,5 +4,5 @@
         <parent link="chassis_link"/>
         <child link="laser_frame"/>
-        <origin xyz="-0.1 0 0.1" rpy="0 0 0"/>
+        <origin xyz="0 0 0.15" rpy="0 0 0"/>
     </joint>
     <link name="laser_frame">
@@ -11,5 +11,5 @@
                 <cylinder length="0.04" radius="0.05"/>
             </geometry>
-            <material name="red"/>
+            <material name="black"/>
         </visual>
         <collision>

File: description/robot_core.xacro (robot description, xacro)
@@ -9,5 +9,5 @@
   <xacro:property name="wheelbase" value="0.289" />
   <xacro:property name="wheel_mass" value="0.34055" /> <!-- arbitrary value for wheel mass -->
-  <xacro:property name="wheel_len" value="0.045" />
+  <xacro:property name="wheel_len" value="0.055" />
   <xacro:property name="wheel_radius" value="0.05" />
   <!-- <xacro:property name="wheeltrack" value="" -->
@@ -34,5 +34,5 @@
         <box size="${base_length} ${base_width} ${base_height}"/>
       </geometry>
-      <material name="orange"/>
+      <material name="green"/>
     </visual>
     <xacro:inertial_box mass="${base_mass}" x="${wheelbase}" y="${base_width}" z="${base_height}">

File: description/ros2_bicycle.xacro (robot description, xacro)
@@ -13,6 +13,6 @@
     <joint name="virtual_rear_wheel_joint">
       <command_interface name="velocity">
-        <param name = "min">-15.5</param>
-        <param name = "max">15.5</param>
+        <param name = "min">-1.0</param>
+        <param name = "max">1.0</param>
       </command_interface>
       <state_interface name="velocity"/>
