Commit message: new xacro for robot_core

File: description/robot_core.xacro (robot description, xacro)
@@ -1,105 +1,103 @@
 <?xml version="1.0"?>
 <robot xmlns:xacro="http://www.ros.org/wiki/xacro"  >
+<!-- A simple model of the racecar for rviz -->
     <xacro:include filename="robot_colors.xacro" />
-    <xacro:include filename="inertial_macros.xacro" />
-    <!-- BASE LINK -->
-    <link name="base_link">
-    </link>
-    <!-- CHASSIS -->
-    <joint name="chassis_joint" type="fixed">
+  <robot xmlns:xacro="http://www.ros.org/wiki/xacro" name="racecar">
+      <xacro:property name="wheelbase" value="0.289" />
+      <xacro:property name="width" value="0.311" />
+      <xacro:property name="height" value="0.178" />
+      <xacro:property name="ground_offset" value="0.04" /> <!--Measure this-->
+      <xacro:property name="wheel_radius" value="0.0508" /> <!--Measure this-->
+      <xacro:property name="wheel_length" value="0.0381" /> <!--Measure this-->
+      <xacro:property name="laser_distance_from_base_link" value="0.275" /> <!--Measure this-->
+      <xacro:property name="laser_height" value="0.05" /> <!--Measure this-->
+      <xacro:property name="laser_radius" value="0.026" /> <!--Measure this-->
+      <link name="base_link">
+        <visual>
+          <origin xyz="${wheelbase/2} 0 ${ground_offset+height/2}"/>
+          <geometry>
+            <box size="${wheelbase} ${width} ${height}"/>
+          </geometry>
+          <material name="orange"/>
+        </visual>
+      </link>
+      <joint name="base_to_laser_model" type="fixed">
         <parent link="base_link"/>
-        <child link="chassis"/>
-        <origin xyz="-0.1 0 0"/>
-    </joint>
-    <link name="chassis">
+        <child link="laser_model"/>
+        <origin xyz="${laser_distance_from_base_link} 0 ${ground_offset+height+(laser_height/2)}"/>
+      </joint>
+      <link name="laser_model">
         <visual>
-            <origin xyz="0.2305 0 0.089"/>
-            <geometry>
-                <box size="0.461 0.311 0.178"/>
-            </geometry>
-            <material name="white"/>
+          <geometry>
+            <cylinder radius="${laser_radius}" length="${laser_height}"/>
+          </geometry>
+          <material name="black"/>
         </visual>
-        <collision>
-            <origin xyz="0.2305 0 0.089" rpy="0 0 0"/>
-            <geometry>
-                <box size="0.461 0.311 0.178"/>
-            </geometry>
-        </collision>
-        <xacro:inertial_box mass="1.69" x="0.461" y="0.311" z="0.178">
-            <origin xyz="0.2305 0 0.089" rpy="0 0 0"/>
-        </xacro:inertial_box>
-    </link>
-    <!-- LEFT DRIVE WHEEL  -->
-    <joint name="left_wheel_joint" type="continuous">
+      </link>
+      <joint name="base_to_back_left_wheel" type="fixed">
         <parent link="base_link"/>
-        <child link="left_wheel"/>
-        <origin xyz="0 0.175 0" rpy="-${pi/2} 0 0"/>
-        <axis xyz="0 0 1"/>
-    </joint>
-    <link name="left_wheel">
+        <child link="back_left_wheel"/>
+        <origin xyz="0 ${(wheel_length+width)/2} ${wheel_radius}"/>
+      </joint>
+      <link name="back_left_wheel">
         <visual>
-            <geometry>
-                <cylinder length="0.04" radius="0.05" />
-            </geometry>
-            <material name="orange"/>
+          <geometry>
+            <cylinder radius="${wheel_radius}" length="${wheel_length}"/>
+          </geometry>
+          <material name="black"/>
+          <origin rpy="${pi/2} 0 0"/>
         </visual>
-        <collision>
-            <geometry>
-                <cylinder length="0.04" radius="0.05" />
-            </geometry>
-        </collision>
-        <!--NEED TO MEASURE PARAMETERS FOR WHEELS AND UPDATE-->
-        <xacro:inertial_cylinder mass="0.1" length="0.04" radius="0.05">
-            <origin xyz="0 0 0" rpy="0 0 0"/>
-        </xacro:inertial_cylinder>
-    </link>
-    <!-- RIGHT DRIVE WHEEL -->
-    <joint name="right_wheel_joint" type="continuous">
+      </link>
+      <joint name="base_to_back_right_wheel" type="fixed">
         <parent link="base_link"/>
-        <child link="right_wheel"/>
-        <origin xyz="0 -0.175 0" rpy="${pi/2} 0 0"/>
-        <axis xyz="0 0 -1"/>
-    </joint>
-    <link name="right_wheel">
+        <child link="back_right_wheel"/>
+        <origin xyz="0 ${-(wheel_length+width)/2} ${wheel_radius}"/>
+      </joint>
+      <link name="back_right_wheel">
         <visual>
-            <geometry>
-                <cylinder length="0.04" radius="0.05" />
-            </geometry>
-            <material name="orange"/>
+          <geometry>
+            <cylinder radius="${wheel_radius}" length="${wheel_length}"/>
+          </geometry>
+          <material name="black"/>
+          <origin rpy="${pi/2} 0 0"/>
         </visual>
-        <collision>
-            <geometry>
-                <cylinder length="0.04" radius="0.05" />
-            </geometry>
-        </collision>
-        <!--NEED TO MEASURE PARAMETERS FOR WHEELS AND UPDATE-->
-        <xacro:inertial_cylinder mass="0.1" length="0.04" radius="0.05">
-            <origin xyz="0 0 0" rpy="0 0 0"/>
-        </xacro:inertial_cylinder>
-    </link>
-    <!-- CASTER WHEEL -->
-    <!-- CREATE TWO CASTER WHEELS LATER-->
-    <joint name="caster_wheel_joint" type="fixed">
-        <parent link="chassis"/>
-        <child link="caster_wheel"/>
-        <origin xyz="0.24 0 0" rpy="0 0 0"/>
-    </joint>
-    <!--UPDATE THIS TO CYLINDER ONCE PARAMETERS FOR WHEELS IS MEASURED-->
-    <link name="caster_wheel">
+      </link>
+      <joint name="base_to_front_left_hinge" type="fixed">
+        <parent link="base_link"/>
+        <child link="front_left_hinge"/>
+        <origin xyz="${wheelbase} ${(wheel_length+width)/2} ${wheel_radius}"/>
+      </joint>
+      <link name="front_left_hinge"/>
+      <joint name="front_left_hinge_to_wheel" type="continuous">
+        <parent link="front_left_hinge"/>
+        <child link="front_left_wheel"/>
+      </joint>
+      <link name="front_left_wheel">
         <visual>
-            <geometry>
-                <sphere radius="0.05" />
-            </geometry>
-            <material name="orange"/>
+          <geometry>
+            <cylinder radius="${wheel_radius}" length="${wheel_length}"/>
+          </geometry>
+          <material name="black"/>
+          <origin rpy="${pi/2} 0 0"/>
         </visual>
-        <collision>
-            <geometry>
-                <sphere radius="0.05" />
-            </geometry>
-        </collision>
-        <!--UPDATE THIS TO CYLINDER ONCE PARAMETERS FOR WHEELS IS MEASURED-->
-        <xacro:inertial_sphere mass="0.1" radius="0.05">
-            <origin xyz="0 0 0" rpy="0 0 0"/>
-        </xacro:inertial_sphere>
-    </link>
+      </link>
+      <joint name="base_to_front_right_hinge" type="fixed">
+        <parent link="base_link"/>
+        <child link="front_right_hinge"/>
+        <origin xyz="${wheelbase} ${-(wheel_length+width)/2} ${wheel_radius}"/>
+      </joint>
+      <link name="front_right_hinge"/>
+      <joint name="front_right_hinge_to_wheel" type="continuous">
+        <parent link="front_right_hinge"/>
+        <child link="front_right_wheel"/>
+      </joint>
+      <link name="front_right_wheel">
+        <visual>
+          <geometry>
+            <cylinder radius="${wheel_radius}" length="${wheel_length}"/>
+          </geometry>
+          <material name="black"/>
+          <origin rpy="${pi/2} 0 0"/>
+        </visual>
+      </link>
 </robot>

Commit message: new robot urdf with ackermann

File: description/robot_core.xacro (robot description, xacro)
@@ -1,103 +1,425 @@
 <?xml version="1.0"?>
-<robot xmlns:xacro="http://www.ros.org/wiki/xacro"  >
-<!-- A simple model of the racecar for rviz -->
-    <xacro:include filename="robot_colors.xacro" />
-  <robot xmlns:xacro="http://www.ros.org/wiki/xacro" name="racecar">
-      <xacro:property name="wheelbase" value="0.289" />
-      <xacro:property name="width" value="0.311" />
-      <xacro:property name="height" value="0.178" />
-      <xacro:property name="ground_offset" value="0.04" /> <!--Measure this-->
-      <xacro:property name="wheel_radius" value="0.0508" /> <!--Measure this-->
-      <xacro:property name="wheel_length" value="0.0381" /> <!--Measure this-->
-      <xacro:property name="laser_distance_from_base_link" value="0.275" /> <!--Measure this-->
-      <xacro:property name="laser_height" value="0.05" /> <!--Measure this-->
-      <xacro:property name="laser_radius" value="0.026" /> <!--Measure this-->
-      <link name="base_link">
-        <visual>
-          <origin xyz="${wheelbase/2} 0 ${ground_offset+height/2}"/>
-          <geometry>
-            <box size="${wheelbase} ${width} ${height}"/>
-          </geometry>
-          <material name="orange"/>
-        </visual>
-      </link>
-      <joint name="base_to_laser_model" type="fixed">
-        <parent link="base_link"/>
-        <child link="laser_model"/>
-        <origin xyz="${laser_distance_from_base_link} 0 ${ground_offset+height+(laser_height/2)}"/>
-      </joint>
-      <link name="laser_model">
-        <visual>
-          <geometry>
-            <cylinder radius="${laser_radius}" length="${laser_height}"/>
-          </geometry>
-          <material name="black"/>
-        </visual>
-      </link>
-      <joint name="base_to_back_left_wheel" type="fixed">
-        <parent link="base_link"/>
+<robot xmlns:xacro="http://ros.org/wiki/xacro" name="car">
+    <xacro:arg name="wheel_diameter" default="0.14224"/>
+    <xacro:property name="wheel_radius" value="${$(arg wheel_diameter)/2}"/>
+    <xacro:property name="wheel_width" value="0.047"/>
+    <xacro:property name="wheel_friction" value="0.8"/>
+    <xacro:property name="wheelbase_length" value="0.311"/>
+    <xacro:property name="front_wheelbase_width" value="0.289"/>
+    <xacro:property name="rear_wheelbase_width" value="0.289"/>
+    <xacro:property name="wheel_mass" value="0.1"/>
+    <xacro:property name="total_mass" value = "3.0"/>
+    <xacro:property name="shock_travel" value = "0.09"/>
+    <xacro:property name="chassis_height" value = "0.178"/>
+    <xacro:property name="chassis_elevation" value = "-0.01"/>
+    <xacro:property name="chassis_mass" value = "${total_mass-4*wheel_mass}"/>
+    <xacro:macro name="cylinder_inertia" params="m r h">
+            <inertia  ixx="${m*(3*r*r+h*h)/12}" ixy = "0" ixz = "0"
+                        iyy="${m*(3*r*r+h*h)/12}" iyz = "0"
+                        izz="${m*r*r/2}" />
+    </xacro:macro>
+    <xacro:macro name="box_inertia" params="m x y z">
+            <inertia  ixx="${m*(y*y+z*z)/12}" ixy = "0" ixz = "0"
+                        iyy="${m*(x*x+z*z)/12}" iyz = "0"
+                        izz="${m*(x*x+z*z)/12}" />
+    </xacro:macro>
+    <xacro:macro name="sphere_inertia" params="m r">
+            <inertia  ixx="${2*m*r*r/5}" ixy = "0" ixz = "0"
+                        iyy="${2*m*r*r/5}" iyz = "0"
+                        izz="${2*m*r*r/5}" />
+    </xacro:macro>
+    <xacro:macro name="cylinder_inertial" params="m r h">
+        <inertial>
+        <mass value="${m}"/>
+        <xacro:cylinder_inertia m="${m}" r="${r}" h="${h}"/>
+        </inertial>
+    </xacro:macro>
+    <link name="base_footprint"/>
+    <link name="base_link"/>
+    <!--
+    <link name="base_link">
+        <visual>
+        <origin xyz="0 0 0.1" rpy="0 0 0"/>
+        <geometry>
+            <cylinder length="0.2" radius="0.01"/>
+        </geometry>
+        <material name="silver">
+            <color rgba="0.75 0.75 0.75 1"/>
+        </material>
+        </visual>
+        <collision>
+        <origin xyz="0 0 0.1" rpy="0 0 0"/>
+        <geometry>
+            <cylinder length="0.2" radius="0.01"/>
+        </geometry>
+        </collision>
+        <inertial>
+        <mass value="0.01"/>
+        <inertia ixx="0.015" iyy="0.0375" izz="0.0375"
+                ixy="0" ixz="0" iyz="0"/>
+        </inertial>
+    </link>
+    -->
+    <link name="chassis_link">
+        <visual>
+        <geometry>
+            <box size="${wheelbase_length} ${front_wheelbase_width} ${chassis_height}"/>
+        </geometry>
+        </visual>
+        <collision>
+        <geometry>
+            <box size="${wheelbase_length} ${front_wheelbase_width} ${chassis_height}"/>
+        </geometry>
+        </collision>
+        <inertial>
+        <mass value="${chassis_mass}"/>
+        <xacro:box_inertia m="${chassis_mass}" x="${wheelbase_length}" y="${front_wheelbase_width}" z="${chassis_height}"/>
+        </inertial>
+    </link>
+    <link name="back_left_wheel">
+        <visual>
+        <geometry>
+            <cylinder length="${wheel_width}" radius="${wheel_radius}"/>
+        </geometry>
+        <material name="black">
+            <color rgba="0 0 0 1"/>
+        </material>
+        </visual>
+        <collision>
+        <geometry>
+            <cylinder length="${wheel_width}" radius="${wheel_radius}"/>
+        </geometry>
+        </collision>
+        <xacro:cylinder_inertial m="${wheel_mass}" r="${wheel_radius}" h="${wheel_width}"/>
+    </link>
+    <link name="laser_scanner_link">
+        <collision>
+        <origin xyz="0 0 0" rpy="0 0 0"/>
+        <geometry>
+            <box size=".127 0.1016 0.0508"/>
+        </geometry>
+        </collision>
+        <visual>
+        <origin xyz="0 0 0" rpy="0 0 0"/>
+        <geometry>
+            <box size=".127 0.1016 0.0508"/>
+        </geometry>
+        </visual>
+        <inertial>
+        <mass value="1e-5"/>
+        <origin xyz="0 0 0" rpy="0 0 0"/>
+        <inertia ixx="1e-6" ixy="0" ixz="0" iyy="1e-6" iyz="0" izz="1e-6"/>
+        </inertial>
+    </link>
+    <gazebo reference="laser_scanner_link">
+        <sensor type="ray" name="laser_scanner">
+        <always_on>true</always_on>
+        <!-- <visualize>true</visualize> -->
+        <update_rate>3</update_rate>
+        <ray>
+        <scan>
+            <horizontal>
+            <samples>360</samples>
+            <resolution>1</resolution>
+            <min_angle>${-pi}</min_angle>
+            <max_angle>${pi}</max_angle>
+            </horizontal>
+        </scan>
+        <range>
+            <min>0.30</min>
+            <max>25.0</max>
+            <resolution>0.1</resolution>
+        </range>
+        </ray>
+        <plugin name="scan" filename="libgazebo_ros_ray_sensor.so">
+            <ros>
+            <remapping>~/out:=scan</remapping>
+            </ros>
+            <output_type>sensor_msgs/LaserScan</output_type>
+            <frame_name>laser_scanner_link</frame_name>
+        </plugin>
+        </sensor>
+    </gazebo>
+    <link name="back_right_wheel">
+        <visual>
+        <geometry>
+            <cylinder length="${wheel_width}" radius="${wheel_radius}"/>
+        </geometry>
+        <material name="black">
+            <color rgba="0 0 0 1"/>
+        </material>
+        </visual>
+        <collision>
+        <geometry>
+            <cylinder length="${wheel_width}" radius="${wheel_radius}"/>
+        </geometry>
+        </collision>
+        <xacro:cylinder_inertial m="${wheel_mass}" r="${wheel_radius}" h="${wheel_width}"/>
+    </link>
+    <link name="front_left_wheel_steer">
+        <visual>
+        <geometry>
+            <cylinder length="0.01" radius="0.01"/>
+        </geometry>
+        <material name="black">
+            <color rgba="0 0 0 1"/>
+        </material>
+        </visual>
+        <collision>
+        <geometry>
+            <cylinder length="0.01" radius="0.01"/>
+        </geometry>
+        </collision>
+        <inertial>
+        <mass value="0.1"/>
+        <inertia ixx="5.1458e-5" iyy="5.1458e-5" izz="6.125e-5"
+                ixy="0" ixz="0" iyz="0"/>
+        </inertial>
+    </link>
+        <link name="front_left_wheel">
+        <visual>
+        <geometry>
+            <cylinder length="${wheel_width}" radius="${wheel_radius}"/>
+        </geometry>
+        <material name="black">
+            <color rgba="0 0 0 1"/>
+        </material>
+        </visual>
+        <collision>
+        <geometry>
+            <cylinder length="${wheel_width}" radius="${wheel_radius}"/>
+        </geometry>
+        </collision>
+        <xacro:cylinder_inertial m="${wheel_mass}" r="${wheel_radius}" h="${wheel_width}"/>
+    </link>
+    <link name="front_right_wheel_steer">
+        <visual>
+        <geometry>
+            <cylinder length="0.01" radius="0.01"/>
+        </geometry>
+        <material name="black">
+            <color rgba="0 0 0 1"/>
+        </material>
+        </visual>
+        <collision>
+        <geometry>
+            <cylinder length="0.01" radius="0.01"/>
+        </geometry>
+        </collision>
+        <inertial>
+        <mass value="0.1"/>
+        <inertia ixx="5.1458e-5" iyy="5.1458e-5" izz="6.125e-5"
+                ixy="0" ixz="0" iyz="0"/>
+        </inertial>
+    </link>
+    <link name="front_right_wheel">
+        <visual>
+        <geometry>
+            <cylinder length="${wheel_width}" radius="${wheel_radius}"/>
+        </geometry>
+        <material name="black">
+            <color rgba="0 0 0 1"/>
+        </material>
+        </visual>
+        <collision>
+        <geometry>
+            <cylinder length="${wheel_width}" radius="${wheel_radius}"/>
+        </geometry>
+        </collision>
+        <xacro:cylinder_inertial m="${wheel_mass}" r="${wheel_radius}" h="${wheel_width}"/>
+    </link>
+    <link name="back_left_wheel_shock">
+        <visual>
+        <origin xyz="0 0 0.1" rpy="0 0 0"/>
+        <geometry>
+            <cylinder length="0.05" radius="0.01"/>
+        </geometry>
+        <material name="silver">
+            <color rgba="0.75 0.75 0.75 1"/>
+        </material>
+        </visual>
+        <collision>
+        <origin xyz="0 0 0.1" rpy="0 0 0"/>
+        <geometry>
+            <cylinder length="0.05" radius="0.01"/>
+        </geometry>
+        </collision>
+        <inertial>
+        <mass value="0.01"/>
+        <inertia ixx="0.015" iyy="0.0375" izz="0.0375"
+                ixy="0" ixz="0" iyz="0"/>
+        </inertial>
+    </link>
+    <link name="back_right_wheel_shock">
+        <visual>
+        <origin xyz="0 0 0.1" rpy="0 0 0"/>
+        <geometry>
+        <cylinder length="0.05" radius="0.01"/>
+        </geometry>
+        <material name="silver">
+        <color rgba="0.75 0.75 0.75 1"/>
+        </material>
+    </visual>
+    <collision>
+        <origin xyz="0 0 0.1" rpy="0 0 0"/>
+        <geometry>
+        <cylinder length="0.05" radius="0.01"/>
+        </geometry>
+    </collision>
+    <inertial>
+        <mass value="0.01"/>
+        <inertia ixx="0.015" iyy="0.0375" izz="0.0375"
+                ixy="0" ixz="0" iyz="0"/>
+    </inertial>
+    </link>
+    <link name="front_left_wheel_shock">
+        <visual>
+        <origin xyz="0 0 0.1" rpy="0 0 0"/>
+        <geometry>
+            <cylinder length="0.05" radius="0.01"/>
+        </geometry>
+        <material name="silver">
+            <color rgba="0.75 0.75 0.75 1"/>
+        </material>
+        </visual>
+        <collision>
+        <origin xyz="0 0 0.1" rpy="0 0 0"/>
+        <geometry>
+            <cylinder length="0.05" radius="0.01"/>
+        </geometry>
+        </collision>
+        <inertial>
+        <mass value="0.01"/>
+        <inertia ixx="0.015" iyy="0.0375" izz="0.0375"
+                ixy="0" ixz="0" iyz="0"/>
+        </inertial>
+    </link>
+    <link name="front_right_wheel_shock">
+        <visual>
+        <origin xyz="0 0 0.1" rpy="0 0 0"/>
+        <geometry>
+            <cylinder length="0.05" radius="0.01"/>
+        </geometry>
+        <material name="silver">
+            <color rgba="0.75 0.75 0.75 1"/>
+        </material>
+        </visual>
+        <collision>
+        <origin xyz="0 0 0.1" rpy="0 0 0"/>
+        <geometry>
+            <cylinder length="0.05" radius="0.01"/>
+        </geometry>
+        </collision>
+        <inertial>
+        <mass value="0.01"/>
+        <inertia ixx="0.015" iyy="0.0375" izz="0.0375"
+                ixy="0" ixz="0" iyz="0"/>
+        </inertial>
+    </link>
+    <joint name="base_link_joint" type="fixed">
+        <parent link="base_footprint"/>
+        <child link="base_link"/>
+        <origin rpy="0 0 0" xyz="0 0 0"/>
+    </joint>
+    <joint name="laser_scanner_joint" type="fixed">
+        <origin rpy="0 0 0" xyz="0.1397 0 0.2159"/>
+        <parent link="base_link"/>
+        <child link="laser_scanner_link"/>
+    </joint>
+    <joint name="back_left_shock_joint" type="prismatic">
+        <limit lower="0" upper="${shock_travel}" effort="100" velocity="100"/>
+        <axis xyz="0 0 1"/>
+        <parent link="base_link"/>
+        <child link="back_left_wheel_shock"/>
+        <origin rpy="0 0 0" xyz="0 ${rear_wheelbase_width/2}  ${-shock_travel/2}"/>
+    </joint>
+    <joint name="back_left_wheel_joint" type="continuous">
+        <axis xyz="0 0 1"/>
+        <parent link="back_left_wheel_shock"/>
         <child link="back_left_wheel"/>
-        <origin xyz="0 ${(wheel_length+width)/2} ${wheel_radius}"/>
-      </joint>
-      <link name="back_left_wheel">
-        <visual>
-          <geometry>
-            <cylinder radius="${wheel_radius}" length="${wheel_length}"/>
-          </geometry>
-          <material name="black"/>
-          <origin rpy="${pi/2} 0 0"/>
-        </visual>
-      </link>
-      <joint name="base_to_back_right_wheel" type="fixed">
-        <parent link="base_link"/>
+        <origin rpy="${-pi/2} 0 0" xyz="0 0 0"/>
+        <limit effort="10000" velocity="500" />
+    </joint>
+    <joint name="back_right_shock_joint" type="prismatic">
+        <limit lower="0" upper="${shock_travel}" effort="100" velocity="100"/>
+        <axis xyz="0 0 1"/>
+        <parent link="base_link"/>
+        <child link="back_right_wheel_shock"/>
+        <origin rpy="0 0 0" xyz="0 ${-rear_wheelbase_width/2} ${-shock_travel/2}"/>
+    </joint>
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