Commit message: Edited Bicycle Steering Controller for debugging

File: description/robot_core.xacro (robot description, xacro)
@@ -29,12 +29,4 @@
       <material name="orange"/>
     </visual>
-    <!-- <inertial>
-      <origin xyz="0 0 0" rpy="0 0 0"/>
-      <mass value="${base_mass}"/>
-        <inertia
-          ixx="0.000270" ixy="0.0" ixz="0.0"
-          iyy="0.000270" iyz="0.0"
-          izz="0.000426"/>
-      </inertial> -->
     <xacro:inertial_box mass="${base_mass}" x="${wheelbase}" y="${base_width}" z="${base_height}">
       <origin xyz="0 0 0" rpy="0 0 0"/>
@@ -88,12 +80,4 @@
         <material name="black"/>
       </visual>
-      <!-- <inertial>
-        <origin xyz="0 0 0" rpy="${PI/2} 0 ${PI/2}"/>
-        <mass value="${wheel_mass}"/>
-        <inertia
-          ixx="0.000270" ixy="0.0" ixz="0.0"
-          iyy="0.000270" iyz="0.0"
-          izz="0.000426"/>
-      </inertial> -->
       <xacro:inertial_cylinder mass="${wheel_mass}" length="${wheel_len}" radius="${wheel_radius}">
           <origin xyz="0 0 0" rpy="${PI/2} 0 ${PI/2}"/>
@@ -127,12 +111,4 @@
           <material name="black"/>
         </visual>
-        <!-- <inertial>
-          <origin xyz="0 0 0" rpy="${PI/2} 0 ${PI/2}"/>
-          <mass value="${wheel_mass}"/>
-          <inertia
-            ixx="0.000270" ixy="0.0" ixz="0.0"
-            iyy="0.000270" iyz="0.0"
-            izz="0.000426"/>
-        </inertial> -->
       <xacro:inertial_cylinder mass="${wheel_mass}" length="${wheel_len}" radius="${wheel_radius}">
           <origin xyz="0 0 0" rpy="${PI/2} 0 ${PI/2}"/>
@@ -188,12 +164,4 @@
         <material name="black"/>
       </visual>
-      <!-- <inertial>
-        <origin xyz="0 0 0" rpy="${PI/2} 0 ${PI/2}"/>
-        <mass value="${wheel_mass}"/>
-        <inertia
-          ixx="0.000270" ixy="0.0" ixz="0.0"
-          iyy="0.000270" iyz="0.0"
-          izz="0.000426"/>
-      </inertial> -->
       <xacro:inertial_cylinder mass="${wheel_mass}" length="${wheel_len}" radius="${wheel_radius}">
           <origin xyz="0 0 0" rpy="${PI/2} 0 ${PI/2}"/>
@@ -227,12 +195,4 @@
         <material name="black"/>
       </visual>
-      <!-- <inertial>
-        <origin xyz="0 0 0" rpy="${PI/2} 0 ${PI/2}"/>
-        <mass value="${wheel_mass}"/>
-        <inertia
-          ixx="0.000270" ixy="0.0" ixz="0.0"
-          iyy="0.000270" iyz="0.0"
-          izz="0.000426"/>
-      </inertial> -->
       <xacro:inertial_cylinder mass="${wheel_mass}" length="${wheel_len}" radius="${wheel_radius}">
           <origin xyz="0 0 0" rpy="${PI/2} 0 ${PI/2}"/>

Commit message: Added base_footprint for sl

File: description/robot_core.xacro (robot description, xacro)
@@ -14,4 +14,11 @@
   <!-- Base Link -->
   <link name="base_link" />
+  <!-- Base Footprint -->
+  <joint name="base_footprint_joint" type="fixed">
+    <parent link="base_link"/>
+    <child link="base_footprint"/>
+    <origin xyz="0 0 0" rpy="0 0 0"/>
+  </joint>
+  <link name="base_footprint" />
   <!-- Chassis -->
   <link name="chassis_link">

Commit message: test

File: description/robot_core.xacro (robot description, xacro)
@@ -7,5 +7,5 @@
   <xacro:property name="base_length" value="0.525" />
   <xacro:property name="base_height" value="0.060" />
-  <xacro:property name="wheelbase" value="0.325" />
+  <xacro:property name="wheelbase" value="0.289" />
   <xacro:property name="wheel_mass" value="0.34055" /> <!-- arbitrary value for wheel mass -->
   <xacro:property name="wheel_len" value="0.045" />

Commit message: updates

File: description/robot_core.xacro (robot description, xacro)
@@ -24,5 +24,5 @@
   <link name="chassis_link">
     <collision>
-      <origin xyz="0 0 0" rpy="0 0 0"/>
+      <origin xyz="${wheelbase/2} 0 ${base_height/2 + wheel_radius}" rpy="0 0 0"/>
       <geometry>
         <box size="${base_length} ${base_width} ${base_height}"/>
@@ -37,14 +37,11 @@
     </visual>
     <xacro:inertial_box mass="${base_mass}" x="${wheelbase}" y="${base_width}" z="${base_height}">
-      <origin xyz="0 0 0" rpy="0 0 0"/>
+      <origin xyz="${wheelbase/2} 0 ${base_height/2 + wheel_radius}" rpy="0 0 0"/>
     </xacro:inertial_box>
     </link>
-    <gazebo reference="chassis_link">
-        <material>Gazebo/Black</material>
-    </gazebo>
     <joint name="chassis_joint" type="fixed">
       <parent link="base_link"/>
       <child link="chassis_link"/>
-      <origin xyz="0 0 ${base_height/2 + wheel_radius}" rpy="0 0 0"/>
+      <origin xyz="${wheelbase/2} 0 ${base_height/2 + wheel_radius}" rpy="0 0 0"/>
       <axis xyz="0 0 1"/>
       <dynamics damping="0.2"/>
@@ -61,7 +58,4 @@
       </visual>
     </link>
-    <gazebo reference="virtual_rear_wheel">
-        <material>Gazebo/White</material>
-    </gazebo>
     <joint name="virtual_rear_wheel_joint" type="continuous">
       <parent link="chassis_link"/>
@@ -91,7 +85,4 @@
       </xacro:inertial_cylinder>
     </link>
-    <gazebo reference="rear_right_wheel">
-        <material>Gazebo/Orange</material>
-    </gazebo>
     <joint name="rear_right_wheel_joint" type="continuous">
       <parent link="chassis_link"/>
@@ -122,7 +113,4 @@
       </xacro:inertial_cylinder>
     </link>
-    <gazebo reference="rear_left_wheel">
-        <material>Gazebo/Orange</material>
-    </gazebo>
     <joint name="rear_left_wheel_joint" type="continuous">
       <parent link="chassis_link" />
@@ -145,7 +133,4 @@
       </visual>
     </link>
-    <gazebo reference="virtual_front_wheel">
-        <material>Gazebo/Black</material>
-    </gazebo>
     <joint name="virtual_front_wheel_joint" type="revolute">
       <parent link="chassis_link"/>
@@ -153,5 +138,5 @@
       <origin xyz="${wheelbase/2} 0 -${base_height/2}" rpy="0 0 ${PI/2}"/>
       <axis xyz="0 0 1"/>
-      <limit lower="-0.4" upper="0.4" effort="100.0" velocity="0.0"/>
+      <limit lower="-0.785398" upper="0.785398" effort="1" velocity="1"/>
       <dynamics damping="0.2"/>
     </joint>
@@ -175,7 +160,4 @@
       </xacro:inertial_cylinder>
     </link>
-    <gazebo reference="front_right_wheel">
-        <material>Gazebo/Orange</material>
-    </gazebo>
     <joint name="front_right_wheel_joint" type="revolute">
       <parent link="chassis_link" />
@@ -183,7 +165,7 @@
       <origin xyz="${wheelbase/2} ${base_width/2} -${base_height/2}" rpy="0 0 ${PI/2}"/>
       <axis xyz="0 0 1"/>
-      <limit lower="-0.4" upper="0.4" effort="100.0" velocity="0.0"/>
+      <limit lower="-0.785398" upper="0.785398" effort="1" velocity="1"/>
       <dynamics damping="0.2"/>
-      <mimic joint="virtual_front_wheel_joint" multiplier="1.0" offset="0.0"/>
+      <!-- <mimic joint="virtual_front_wheel_joint" multiplier="1.0" offset="0.0"/> -->
     </joint>
     <!-- front left steering -->
@@ -206,7 +188,4 @@
       </xacro:inertial_cylinder>
     </link>
-    <gazebo reference="front_left_wheel">
-        <material>Gazebo/Orange</material>
-    </gazebo>
     <joint name="front_left_wheel_joint" type="revolute">
       <parent link="chassis_link" />
@@ -214,7 +193,7 @@
       <origin xyz="${wheelbase/2} -${base_width/2} -${base_height/2}" rpy="0 0 ${PI/2}"/>
       <axis xyz="0 0 1"/>
-      <limit lower="-0.4" upper="0.4" effort="100.0" velocity="0.0"/>
+      <limit lower="-0.785398" upper="0.785398" effort="1" velocity="1"/>
       <dynamics damping="0.2"/>
-      <mimic joint="virtual_front_wheel_joint" multiplier="1.0" offset="0.0"/>
+      <!-- <mimic joint="virtual_front_wheel_joint" multiplier="0.5" offset="0.0"/> -->
     </joint>
 </robot>

Commit message: Final Updates

File: description/robot_core.xacro (robot description, xacro)
@@ -63,5 +63,5 @@
       <origin xyz="-${wheelbase/2} 0 -${base_height/2}" rpy="0 0 ${PI/2}"/>
       <axis xyz="1 0 0"/>
-      <limit effort="100.0" velocity="100.0"/>
+      <limit effort="100.0" velocity="0.5"/>
       <dynamics damping="0.2"/>
     </joint>
@@ -90,5 +90,5 @@
       <origin xyz="-${wheelbase/2} ${base_width/2} -${base_height/2}" rpy="0 0 ${PI/2}"/>
       <axis xyz="1 0 0"/>
-      <limit effort="100.0" velocity="100.0"/>
+      <limit effort="100.0" velocity="0.5"/>
       <dynamics damping="0.2"/>
       <mimic joint="virtual_rear_wheel_joint" multiplier="1.0" offset="0.0"/>
@@ -118,5 +118,5 @@
       <origin xyz="-${wheelbase/2} -${base_width/2} -${base_height/2}" rpy="0 0 ${PI/2}"/>
       <axis xyz="1 0 0"/>
-      <limit effort="100.0" velocity="100.0"/>
+      <limit effort="100.0" velocity="0.5"/>
       <dynamics damping="0.2"/>
       <mimic joint="virtual_rear_wheel_joint" multiplier="1.0" offset="0.0"/>
